File: 8mbsimm/8MBSIMM.brd (EAGLE design)
At the start: 97.8 x 27.9 mm, 10 parts, among them CON1 MYSIMM, IC1 M29F160FB5AN6E2, IC2 M29F160FB5AN6E2, IC3 M29F160FB5AN6E2, IC4 M29F160FB5AN6E2

Commit message: Changed for final revision: moved jolly roger logo to center.
Parts:
- moved U$1 36.0 mm to (59.2, 7.06)
Other:
- board text added: "61977"
- board text removed: "58179"
Changed lines of the file:
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@@
 <?xml version="1.0" encoding="utf-8"?>
 <!DOCTYPE eagle SYSTEM "eagle.dtd">
-<eagle version="6.2">
+<eagle version="6.3">
 <drawing>
 <settings>
@@
 <board>
 <plain>
-<text x="97.4725" y="21.193125" size="1.27" layer="25" rot="R90">58179</text>
+<text x="97.4725" y="21.193125" size="1.27" layer="25" rot="R90">61977</text>
 </plain>
 <attributes>
@@
 </class>
 </classes>
-<designrules>
+<designrules name="default *">
 <description language="de">&lt;b&gt;EAGLE Design Rules&lt;/b&gt;
 &lt;p&gt;
@@
 <attribute name="VALUE" x="83.915" y="25.375625" size="1.27" layer="27" rot="R270"/>
 </element>
-<element name="U$1" library="Doug" package="JOLLYROGER" value="" x="23.33625" y="9.8425" rot="MR0"/>
+<element name="U$1" library="Doug" package="JOLLYROGER" value="" x="59.21375" y="7.064375" rot="MR0"/>
 </elements>
 <signals>
